File: PCB/PCB.kicad_pcb (KiCad board)
At the start: 2 copper layers, 19.5 x 29.5 mm, 6 parts, among them P1 USB_C_Plug_USB2.0, Q1 BC107

Commit message: Route PCB
Routing:
- net Net-(P1-GND-PadA1): track 0.00 -> 47.5 mm
- net Net-(D1-A): track 0.00 -> 27.7 mm
- net Net-(Q1-B): track 0.00 -> 23.2 mm
- net Net-(Q1-E): track 0.00 -> 22.1 mm
- net Net-(D1-K): track 0.00 -> 8.49 mm
Changed lines of the file:
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@@
 		)
+	)
+	(segment
+		(start 152.5 84.49295)
+		(end 152.5 82)
+		(width 0.2)
+		(layer "F.Cu")
+		(net 1)
+	)
+	(segment
+		(start 160.5 100.5)
+		(end 164.735 100.5)
+		(width 0.2)
+		(layer "F.Cu")
+		(net 1)
+	)
+	(segment
+		(start 154.35 102.32)
+		(end 154.35 86.34295)
+		(width 0.2)
+		(layer "F.Cu")
+		(net 1)
+	)
+	(segment
+		(start 154.35 86.34295)
+		(end 152.5 84.49295)
+		(width 0.2)
+		(layer "F.Cu")
+		(net 1)
+	)
+	(segment
+		(start 159.15 102.32)
+		(end 159.15 101.85)
+		(width 0.2)
+		(layer "F.Cu")
+		(net 1)
+	)
+	(segment
+		(start 159.15 101.85)
+		(end 160.5 100.5)
+		(width 0.2)
+		(layer "F.Cu")
+		(net 1)
+	)
+	(segment
+		(start 167 92.119448)
+		(end 167 100.225)
+		(width 0.2)
+		(layer "B.Cu")
+		(net 2)
+	)
+	(segment
+		(start 167 100.225)
+		(end 167.275 100.5)
+		(width 0.2)
+		(layer "B.Cu")
+		(net 2)
+	)
+	(segment
+		(start 161.272529 100.997471)
+		(end 163.534 100.997471)
+		(width 0.2)
+		(layer "F.Cu")
+		(net 4)
+	)
+	(segment
+		(start 165.936 98.336)
+		(end 160.7 93.1)
+		(width 0.2)
+		(layer "F.Cu")
+		(net 4)
+	)
+	(segment
+		(start 165.936 100.997471)
+		(end 165.936 98.336)
+		(width 0.2)
+		(layer "F.Cu")
+		(net 4)
+	)
+	(segment
+		(start 165.232471 101.701)
+		(end 165.936 100.997471)
+		(width 0.2)
+		(layer "F.Cu")
+		(net 4)
+	)
+	(segment
+		(start 163.534 100.997471)
+		(end 164.237529 101.701)
+		(width 0.2)
+		(layer "F.Cu")
+		(net 4)
+	)
+	(segment
+		(start 159.95 102.32)
+		(end 161.272529 100.997471)
+		(width 0.2)
+		(layer "F.Cu")
+		(net 4)
+	)
+	(segment
+		(start 164.237529 101.701)
+		(end 165.232471 101.701)
+		(width 0.2)
+		(layer "F.Cu")
+		(net 4)
+	)
+	(segment
+		(start 160.7 98.2)
+		(end 160.7 93.1)
+		(width 0.2)
+		(layer "B.Cu")
+		(net 4)
+	)
+	(segment
+		(start 168.476 101.701)
+		(end 164.201 101.701)
+		(width 0.2)
+		(layer "B.Cu")
+		(net 4)
+	)
+	(segment
+		(start 164.201 101.701)
+		(end 160.7 98.2)
+		(width 0.2)
+		(layer "B.Cu")
+		(net 4)
+	)
+	(segment
+		(start 168.476 86.786)
+		(end 168.476 101.701)
+		(width 0.2)
+		(layer "B.Cu")
+		(net 4)
+	)
+	(segment
+		(start 167.74 86.05)
+		(end 168.476 86.786)
+		(width 0.2)
+		(layer "B.Cu")
+		(net 4)
+	)
+	(segment
+		(start 152.64395 94.201)
+		(end 153.55605 94.201)
+		(width 0.2)
+		(layer "B.Cu")
+		(net 8)
+	)
+	(segment
+		(start 163.840552 91.5)
+		(end 164.46 92.119448)
+		(width 0.2)
+		(layer "B.Cu")
+		(net 8)
+	)
+	(segment
+		(start 152.5 86.05)
+		(end 151.700001 86.849999)
+		(width 0.2)
+		(layer "B.Cu")
+		(net 8)
+	)
+	(segment
+		(start 151.700001 93.257051)
+		(end 152.64395 94.201)
+		(width 0.2)
+		(layer "B.Cu")
+		(net 8)
+	)
+	(segment
+		(start 151.700001 86.849999)
+		(end 151.700001 93.257051)
+		(width 0.2)
+		(layer "B.Cu")
+		(net 8)
+	)
+	(segment
+		(start 153.55605 94.201)
+		(end 156.25705 91.5)
+		(width 0.2)
+		(layer "B.Cu")
+		(net 8)
+	)
+	(segment
+		(start 156.25705 91.5)
+		(end 163.840552 91.5)
+		(width 0.2)
+		(layer "B.Cu")
+		(net 8)
+	)
+	(segment
+		(start 155.350552 90.849448)
+		(end 165.73 90.849448)
+		(width 0.2)
+		(layer "B.Cu")
+		(net 9)
+	)
+	(segment
+		(start 167.74 82)
+		(end 165.73 84.01)
+		(width 0.2)
+		(layer "B.Cu")
+		(net 9)
+	)
+	(segment
+		(start 165.73 84.01)
+		(end 165.73 90.849448)
+		(width 0.2)
+		(layer "B.Cu")
+		(net 9)
+	)
+	(segment
+		(start 153.1 93.1)
+		(end 155.350552 90.849448)
+		(width 0.2)
+		(layer "B.Cu")
+		(net 9)
 	)
 	(group ""

Commit message: Clean up board
Parts:
- Q1: value BC107 -> BC549C; footprint Package_TO_SOT_THT:TO-92 -> Package_TO_SOT_THT:TO-92_Inline_Wide
- R1: value R -> 72kΩ
- R2: value LDR03 -> 3k-70kΩ
- R3: value R -> 150Ω
- moved Q1 3.54 mm to (167.0, 94.6), turned to 90 degrees
Routing:
- net Net-(P1-GND-PadA1): track 47.5 -> 29.8 mm
- net Net-(Q1-B): track 23.2 -> 30.5 mm
- net Net-(D1-K): track 8.49 -> 14.4 mm
- net Net-(Q1-E): track 22.1 -> 26.1 mm
- net Net-(D1-A): track 27.7 -> 31.7 mm
