File: PCB/PCB.kicad_pcb (KiCad board)
At the start: 2 copper layers, 30.5 x 24 mm, 6 parts, among them U1 Seeed Studio XIAO SAMD21

Commit message: Revert to malted's PCB
Parts:
- removed U1: Seeed Studio XIAO SAMD21, Custom:XIAO-RP2040-SMD
- added J1: USB_C_Receptacle_PowerOnly_6P, Connector_USB:USB_C_Receptacle_GCT_USB4125-xx-x-0190_6P_TopMnt_Horizontal, F.Cu at (157.5, 105.7)
- added R1: 5k1Ω, Resistor_SMD:R_0402_1005Metric, F.Cu at (155.8, 100.8)
- added R4: 5k1Ω, Resistor_SMD:R_0402_1005Metric, F.Cu at (157.7, 100.9)
- R3: value 68Ω -> 150Ω
- moved D1 19.6 mm to (165.5, 107.0), turned to 90 degrees
- moved R3 15.4 mm to (163.9, 102.8)
- moved RV1 9.85 mm to (155.0, 98.5)
- moved Q1 9.48 mm to (160.6, 98.5), turned to 180 degrees
- moved R2 5.22 mm to (164.3, 100.0)
Routing:
- net Net-(Q1-S): track 17.0 -> 8.79 mm
- net Net-(Q1-G): track 12.3 -> 8.47 mm
- net Net-(J1-CC2): track 0.00 -> 3.18 mm, vias 0 -> 2
- net Net-(J1-SHIELD): track 46.3 -> 43.7 mm, vias 0 -> 3
- net Net-(D1-K): track 18.9 -> 21.5 mm
- net Net-(D1-A): track 23.3 -> 21.3 mm
- net Net-(J1-CC1): track 0.00 -> 1.83 mm
Other:
- board size 30.5 x 24 mm -> 18 x 13 mm
- board text added: "Thing 1 @Malted"
