File: PCB/PCB.kicad_sch (KiCad schematic)
At the start: 6 parts, among them P1 USB_C_Plug_USB2.0, Q1 BC107

Commit message: Add writeups
Parts:
- R1: value R -> ?Ω
- R2: value LDR03 -> 3kΩ
Changed lines of the file:
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@@
 			)
 		)
-		(property "Value" "LDR03"
+		(property "Value" "3kΩ"
 			(at 129.54 81.2799 0)
 			(effects
@@
 			)
 		)
-		(property "Value" "R"
+		(property "Value" "?Ω"
 			(at 129.54 60.9599 0)
 			(effects

Commit message: Clean up board
Parts:
- Q1: value BC107 -> BC549C; footprint Package_TO_SOT_THT:TO-92 -> Package_TO_SOT_THT:TO-92_Inline_Wide
- R1: value ?Ω -> 72kΩ
- R2: value 3kΩ -> 3k-70kΩ
- R3: value R -> 150Ω
Changed lines of the file:
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@@
 			)
 		)
-		(property "Value" "3kΩ"
+		(property "Value" "3k-70kΩ"
 			(at 129.54 81.2799 0)
 			(effects
@@
 			)
 		)
-		(property "Value" "BC107"
+		(property "Value" "BC549C"
 			(at 146.05 71.1199 0)
 			(effects
@@
 			)
 		)
-		(property "Footprint" "Package_TO_SOT_THT:TO-92"
+		(property "Footprint" "Package_TO_SOT_THT:TO-92_Inline_Wide"
 			(at 146.05 71.755 0)
 			(effects
@@
 			)
 		)
-		(property "Value" "R"
+		(property "Value" "150Ω"
 			(at 146.05 83.8199 0)
 			(effects
@@
 			)
 		)
-		(property "Value" "?Ω"
+		(property "Value" "72kΩ"
 			(at 129.54 60.9599 0)
 			(effects

Commit message: Reroute PCB
Parts:
- removed P1: USB_C_Plug_USB2.0, Connector_USB:USB_C_Receptacle_GCT_USB4105-xx-A_16P_TopMnt_Horizontal, symbol Connector:USB_C_Plug_USB2.0
- removed Q1: BC549C, Package_TO_SOT_THT:TO-92_Inline_Wide, symbol Transistor_BJT:BC107
- removed R1: 72kΩ, Resistor_THT:R_Axial_DIN0207_L6.3mm_D2.5mm_P15.24mm_Horizontal, symbol Device:R
- added J1: USB_C_Receptacle_PowerOnly_6P, Connector_USB:USB_C_Receptacle_GCT_USB4125-xx-x-0190_6P_TopMnt_Horizontal, symbol Connector:USB_C_Receptacle_PowerOnly_6P
- added Q1: ~, Package_TO_SOT_SMD:SOT-23, symbol Transistor_FET:T2N7002AK
- added RV1: 100kΩ, Potentiometer_SMD:Potentiometer_Bourns_TC33X_Vertical, symbol Device:R_Potentiometer_Trim
- R2: footprint OptoDevice:R_LDR_10x8.5mm_P7.6mm_Vertical -> OptoDevice:R_LDR_5.1x4.3mm_P3.4mm_Vertical
- R3: footprint Resistor_THT:R_Axial_DIN0207_L6.3mm_D2.5mm_P15.24mm_Horizontal -> Resistor_SMD:R_0402_1005Metric
Connections:
- net at R2.1: now also Q1.1 (G), RV1.2
- net at R2.2, R3.2: now also J1.A12 (GND), J1.B12 (GND), J1.S1 (SHIELD), RV1.3
- net at R3.1: now also Q1.2 (S)
- net at D1.1 (K): now also Q1.3 (D)
- net at D1.2 (A): now also J1.A9 (VBUS), J1.B9 (VBUS), RV1.1
Other:
- moved on the sheet: D1, R3

Commit message: Add 5k1 CC resistors to negotiate 5V
Parts:
- added R1, R4: 5k1Ω, symbol Device:R
Connections:
- net at J1.A12 (GND), J1.B12 (GND), J1.S1 (SHIELD)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: now also R1.2, R4.2
- net at J1.A5 (CC1): now also R4.1
- net at J1.B5 (CC2): now also R1.1
Other:
- moved on the sheet: RV1
Changed lines of the file:
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@@
+	)
+	(junction
+		(at 110.49 88.9)
+		(diameter 0)
+		(color 0 0 0 0)
+	)
+	(junction
+		(at 120.65 69.85)
+		(diameter 0)
+		(color 0 0 0 0)
 	)
 	(junction
@@
 	(wire
 		(pts
-			(xy 120.65 68.58) (xy 120.65 88.9)
+			(xy 120.65 67.31) (xy 120.65 69.85)
+		)
+		(stroke
+			(width 0)
+			(type default)
+		)
+	)
+	(wire
+		(pts
+			(xy 119.38 69.85) (xy 120.65 69.85)
 		)
 		(stroke
@@
 	(wire
 		(pts
-			(xy 120.65 57.15) (xy 120.65 60.96)
+			(xy 120.65 57.15) (xy 120.65 59.69)
+		)
+		(stroke
+			(width 0)
+			(type default)
+		)
+	)
+	(wire
+		(pts
+			(xy 110.49 87.63) (xy 110.49 88.9)
 		)
 		(stroke
@@
 	(wire
 		(pts
-			(xy 124.46 64.77) (xy 127 64.77)
+			(xy 124.46 63.5) (xy 127 63.5)
+		)
+		(stroke
+			(width 0)
+			(type default)
+		)
+	)
+	(wire
+		(pts
+			(xy 110.49 69.85) (xy 111.76 69.85)
+		)
+		(stroke
+			(width 0)
+			(type default)
+		)
+	)
+	(wire
+		(pts
+			(xy 120.65 69.85) (xy 120.65 88.9)
+		)
+		(stroke
+			(width 0)
+			(type default)
+		)
+	)
+	(wire
+		(pts
+			(xy 110.49 88.9) (xy 120.65 88.9)
 		)
 		(stroke
@@
 	(wire
 		(pts
-			(xy 95.25 88.9) (xy 120.65 88.9)
+			(xy 95.25 88.9) (xy 110.49 88.9)
 		)
 		(stroke
@@
 	(wire
 		(pts
-			(xy 127 64.77) (xy 127 72.39)
+			(xy 127 63.5) (xy 127 72.39)
+		)
+		(stroke
+			(width 0)
+			(type default)
+		)
+	)
+	(wire
+		(pts
+			(xy 110.49 72.39) (xy 110.49 80.01)
 		)
 		(stroke
@@
 	)
 	(symbol
+		(lib_id "Device:R")
+		(at 110.49 83.82 0)
+		(unit 1)
+		(exclude_from_sim no)
+		(in_bom yes)
+		(on_board yes)
+		(dnp no)
+		(fields_autoplaced yes)
+		(property "Reference" "R1"
+			(at 113.03 82.5499 0)
+			(effects
+				(font
+					(size 1.27 1.27)
+				)
+				(justify left)
+			)
+		)
+		(property "Value" "5k1Ω"
+			(at 113.03 85.0899 0)
+			(effects
+				(font
+					(size 1.27 1.27)
+				)
+				(justify left)
+			)
+		)
+		(property "Footprint" ""
+			(at 108.712 83.82 90)
+			(effects
+				(font
+					(size 1.27 1.27)
+				)
+				(hide yes)
+			)
+		)
+		(property "Datasheet" "~"
+			(at 110.49 83.82 0)
+			(effects
+				(font
+					(size 1.27 1.27)
+				)
+				(hide yes)
+			)
+		)
+		(property "Description" "Resistor"
+			(at 110.49 83.82 0)
+			(effects
+				(font
+					(size 1.27 1.27)
+				)
+				(hide yes)
+			)
+		)
+		(pin "2"
+		)
+		(pin "1"
+		)
+		(instances
+			(project ""
+				(path "/54a3e53b-4573-43bc-9261-ecb3a85bc71e"
+					(reference "R1")
+					(unit 1)
+				)
+			)
+		)
+	)
+	(symbol
 		(lib_id "Connector:USB_C_Receptacle_PowerOnly_6P")
 		(at 95.25 64.77 0)
@@
 	(symbol
 		(lib_id "Device:R_Potentiometer_Trim")
-		(at 120.65 64.77 0)
+		(at 120.65 63.5 0)
 		(unit 1)
 		(exclude_from_sim no)
@@
 		(on_board yes)
 		(dnp no)
-		(fields_autoplaced yes)
 		(property "Reference" "RV1"
-			(at 118.11 63.4999 0)
+			(at 118.11 62.2299 0)
 			(effects
 				(font
@@
 		)
 		(property "Value" "100kΩ"
-			(at 118.11 66.0399 0)
+			(at 118.364 64.516 0)
 			(effects
 				(font
@@
 		)
 		(property "Footprint" "Potentiometer_SMD:Potentiometer_Bourns_TC33X_Vertical"
-			(at 120.65 64.77 0)
+			(at 120.65 63.5 0)
 			(effects
 				(font
@@
 		)
 		(property "Datasheet" "https://www.bourns.com/docs/Product-Datasheets/TC33.pdf"
-			(at 120.65 64.77 0)
+			(at 120.65 63.5 0)
 			(effects
 				(font
@@
 		)
 		(property "Description" "Trim-potentiometer"
-			(at 120.65 64.77 0)
+			(at 120.65 63.5 0)
 			(effects
 				(font
@@
 					(unit 1)
 				)
+			)
+		)
+	)
+	(symbol
+		(lib_id "Device:R")
+		(at 115.57 69.85 90)
+		(unit 1)
+		(exclude_from_sim no)
+		(in_bom yes)
+		(on_board yes)
+		(dnp no)
+		(property "Reference" "R4"
+			(at 115.57 72.39 90)
+			(effects
+				(font
+					(size 1.27 1.27)
+				)
+			)
+		)
+		(property "Value" "5k1Ω"
+			(at 115.57 74.676 90)
+			(effects
+				(font
+					(size 1.27 1.27)
+				)
+			)
+		)
+		(property "Footprint" ""
+			(at 115.57 71.628 90)
+			(effects
+				(font
+					(size 1.27 1.27)
+				)
+				(hide yes)
+			)
+		)
+		(property "Datasheet" "~"
+			(at 115.57 69.85 0)
+			(effects
+				(font
+					(size 1.27 1.27)
+				)
+				(hide yes)
+			)
+		)
+		(property "Description" "Resistor"
+			(at 115.57 69.85 0)
+			(effects
+				(font
+					(size 1.27 1.27)
+				)
+				(hide yes)
+			)
+		)
+		(pin "1"
+		)
+		(pin "2"
+		)
+		(instances
+			(project ""
+				(path "/54a3e53b-4573-43bc-9261-ecb3a85bc71e"
+					(reference "R4")
+					(unit 1)
+				)

Commit message: Add and route CC 5k1Ω resistors
Parts:
- R1, R4: footprint (none) -> Resistor_SMD:R_0402_1005Metric
Changed lines of the file:
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@@
 			)
 		)
-		(property "Footprint" ""
+		(property "Footprint" "Resistor_SMD:R_0402_1005Metric"
 			(at 108.712 83.82 90)
 			(effects
@@
 			)
 		)
-		(property "Footprint" ""
+		(property "Footprint" "Resistor_SMD:R_0402_1005Metric"
 			(at 115.57 71.628 90)
 			(effects
