File: PCB/thing.kicad_pcb (KiCad board)
At the start: 2 copper layers, 30.5 x 24 mm, 6 parts, among them U1 Seeed Studio XIAO SAMD21

Commit message: Add files via upload
Parts:
- D1: moved to F.Cu
- moved Q1 41.7 mm to (129.0, 91.0), turned to 0 degrees
- moved R2 39.2 mm to (128.3, 83.5)
- moved RV1 35.1 mm to (129.3, 97.0)
- moved R3 30.5 mm to (132.0, 88.0)
- moved D1 14.9 mm to (156.7, 99.0)
- moved U1 7.66 mm to (144.0, 91.9)
Routing:
- net Net-(D1-A): track 23.3 -> 59.8 mm
- net Net-(D1-K): track 18.9 -> 38.2 mm
- net Net-(U1-PA02_A0_D0): track 46.3 -> 33.5 mm
- net Net-(Q1-S): track 17.0 -> 7.85 mm
- net Net-(Q1-G): track 12.3 -> 21.2 mm
Other:
- board size 30.5 x 24 mm -> 36.5 x 24.5 mm
- board text removed: "(symbol "LOGO" (pin_names (offset 1.016)) (in_bom yes) (on_board yes) (property "Reference" "#G" (at 0 16.994 0) (effects (font (size 1.27 1.27)) hide) ) (property "Value" "LOGO" (at 0 -16.994 0) (effects (font (size 1.27 1.27)) hide) ) (property "Footprint" "" (at 0 0 0) (effects (font (size 1.27 1.27)) hide) ) (property "Datasheet" "" (at 0 0 0) (effects (font (size 1.27 1.27)) hide) ) (symbol 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"

Commit message: Add files via upload
Parts:
- D1: moved to B.Cu
