File: PCB/PCB2.kicad_sch (KiCad schematic)
At the start: 8 parts, among them J1 USB_C_Receptacle_PowerOnly_6P

Commit message: Rebuilt PCB
Parts:
- removed R2: 3k-70kΩ, OptoDevice:R_LDR_5.1x4.3mm_P3.4mm_Vertical, symbol Sensor_Optical:LDR03
- removed R4: 5k1Ω, Resistor_SMD:R_0402_1005Metric, symbol Device:R
- added R2: 5k1Ω, Resistor_SMD:R_0402_1005Metric, symbol Device:R
- added R4: 3k-70kΩ, OptoDevice:R_LDR_5.1x4.3mm_P3.4mm_Vertical, symbol Device:R_Photo
- Q1: value ~ -> T2N7002AK
Connections:
- net at Q1.1 (G), RV1.2: now also R4.1
- net at J1.A12 (GND), J1.B12 (GND), J1.S1 (SHIELD)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: now also R2.2, R4.2
- net at J1.A5 (CC1): now also R2.1

Commit message: add my project files
Parts:
- added BZ1: Buzzer, Buzzer_Beeper:Buzzer_12x9.5RM7.6, symbol Device:Buzzer
- added D18, D3, D4, D5, D6: D, ScottoKeebs_Components:Diode_SOD-123, symbol Device:D
- added J2: OLED_128x64, ScottoKeebs_Components:OLED_128x32, symbol ScottoKeebs:OLED_128x32
- added SW1: RotaryEncoder_Switch, ScottoKeebs_Components:RollerEncoder_Panasonic_EVQWGD001, symbol Device:RotaryEncoder_Switch
- added SW3, SW4, SW5, SW6: SW_Push_45deg, MX_Solderable:MX-Solderable-1U, symbol Switch:SW_Push_45deg
- added U2: XIAO-RP2040-DIP, Seeed Studio XIAO Series Library:XIAO-RP2040-DIP, symbol Seeed_Studio_XIAO_Series:XIAO-RP2040-DIP
Connections:
- new net: D5.2 (A), SW5.2
- new net: D6.2 (A), SW6.2
- new net: D4.2 (A), SW4.2
- new net: D18.2 (A), SW1.S2
- new net: D3.2 (A), SW3.2
- new net +5V: J2.2 (VCC), U2.14 (VBUS)
- new net Buzzer: BZ1.1 (+), U2.1 (GPIO26/ADC0/A0)
- new net Column 0: SW3.1, U2.11 (GPIO3/MOSI)
- new net Column 1: SW4.1, U2.10 (GPIO4/MISO)
- new net Column 2: SW5.1, U2.9 (GPIO2/SCK)
- new net Column 3: SW6.1, U2.8 (GPIO1/RX)
- new net Column 4: SW1.S1, U2.7 (GPIO0/TX)
- new net ENCODER A: SW1.A, U2.2 (GPIO27/ADC1/A1)
- new net ENCODER B: SW1.B, U2.3 (GPIO28/ADC2/A2)
- new net GND: BZ1.2 (-), J2.1 (GND), SW1.C, U2.13 (GND)
- new net Row 0: D18.1 (K), D3.1 (K), D4.1 (K), D5.1 (K), D6.1 (K), U2.4 (GPIO29/ADC3/A3)
- new net SCL: J2.3 (SCL), U2.6 (GPIO7/SCL)
- new net SDA: J2.4 (SDA), U2.5 (GPIO6/SDA)
- no-connect marks 0 -> 1
Other:
- note added: "@Malted"
- note added: "@lukas"
- title: (none) -> The Thing
- moved on the sheet: D1, J1, Q1, R1, R2, R3, R4, RV1
